File: 6632B_binding_posts.kicad_sch (KiCad schematic)
At the start: 21 parts, among them J1 Conn_01x01, J615 Conn_01x04_Male

Commit message: Update logo
Parts:
- LOGO1, LOGO2: now left out of the parts list
Changed lines of the file:
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@@
 		(unit 1)
 		(exclude_from_sim yes)
-		(in_bom yes)
+		(in_bom no)
 		(on_board yes)
 		(dnp no)
@@
 		(at 243.84 170.18 0)
 		(unit 1)
-		(exclude_from_sim no)
-		(in_bom yes)
+		(exclude_from_sim yes)
+		(in_bom no)
 		(on_board yes)
 		(dnp no)
